Commit message: Refine D1 rear panel colors and maintain overlapping lift covers

File: src/manipulation_kit/description/d1/d1_wholebody.urdf (robot description, URDF)
Before this commit: robot d1_wholebody, 43 links, 42 joints
Links:
- link chassis_link: geometry collision box size=0.14 0.14 0.5; collision box size=0.5395 0.4805 0.223
- link torso_column: geometry collision box size=0.0323 0.119 0.119; collision box size=0.09 0.11 0.49

File: src/manipulation_kit/description/d1/d1_wholebody_gripper.urdf (robot description, URDF)
Before this commit: robot d1_wholebody_gripper, 45 links, 44 joints
Links:
- link chassis_link: geometry collision box size=0.14 0.14 0.5; collision box size=0.5395 0.4805 0.223
- link torso_column: geometry collision box size=0.0323 0.119 0.119; collision box size=0.09 0.11 0.49

Commit message: Correct D1 controls, white chassis and head shell surfaces

File: src/manipulation_kit/description/d1/d1_wholebody.urdf (robot description, URDF)
Before this commit: robot d1_wholebody, 43 links, 42 joints
Links:
- link chassis_link: geometry collision box size=0.14 0.14 0.5; collision box size=0.5395 0.4805 0.223
- link head_link: geometry collision box size=0.2008 0.185 0.19; visual mesh filename=meshes/body_hifi/head_link_cyan.obj
- link torso_column: geometry collision box size=0.0323 0.119 0.119; collision box size=0.09 0.11 0.49

File: src/manipulation_kit/description/d1/d1_wholebody_gripper.urdf (robot description, URDF)
Before this commit: robot d1_wholebody_gripper, 45 links, 44 joints
Links:
- link chassis_link: geometry collision box size=0.14 0.14 0.5; collision box size=0.5395 0.4805 0.223
- link head_link: geometry collision box size=0.2008 0.185 0.19; visual mesh filename=meshes/body_hifi/head_link_cyan.obj
- link torso_column: geometry collision box size=0.0323 0.119 0.119; collision box size=0.09 0.11 0.49

Commit message: Model gallery chassis apron, caster clearance and slim forehead optics

File: src/manipulation_kit/description/d1/d1_wholebody.urdf (robot description, URDF)
Before this commit: robot d1_wholebody, 43 links, 42 joints
Links:
- link chassis_link: geometry collision box size=0.14 0.14 0.5; collision box size=0.5395 0.4805 0.223
- link head_link: geometry collision box size=0.2008 0.185 0.19; visual mesh filename=meshes/body_hifi/head_link_cyan.obj

File: src/manipulation_kit/description/d1/d1_wholebody_gripper.urdf (robot description, URDF)
Before this commit: robot d1_wholebody_gripper, 45 links, 44 joints
Links:
- link chassis_link: geometry collision box size=0.14 0.14 0.5; collision box size=0.5395 0.4805 0.223
- link head_link: geometry collision box size=0.2008 0.185 0.19; visual mesh filename=meshes/body_hifi/head_link_cyan.obj
