Commit message: Head camera nominal down-tilt: 17.25 deg -> 15 deg (head-part CAD)
The head camera's downward pitch was inferred from the D435 slab normal
(0.955, 0.005, -0.297) in the 2026-08-23 full-robot CAD, giving 17.25 deg.
That was the best source available: the vendor housing mesh the mount is
solved from is an axis-aligned bar, so its AABB carries no tilt.

The head-part CAD section (Shu, 2026-09-17) gives the mounting face
directly: the D435 module sits 15 deg below horizontal, deliberately, so the
field of view is aimed down at the workspace. That is the design value and it
supersedes the slab reading, so HEAD_CAMERA_PITCH is now math.radians(15.0).

Only the rotation changes. The mount translation is still solved from the
housing mesh at generation time, so head_camera_link stays at
(0.0966561, -0.0732024, -0.0282995) in head_link and 1.2627 m above the floor
at the lift origin. The whole-body URDFs are regenerated, not edited: the
only functional line that moves is head_camera_mount rpy, 0.301131 ->
0.261799. d1.urdf carries no cameras and is untouched.

Still nominal, and the comment now says so with a number. The d1-3 head ArUco
calibration (d1-inference calibrate_head_aruco.py, session
d1-3-tokyo-20260916, neck sweep) reads the optical axis 12.2-12.8 deg below
head_link forward with -1.3...-1.9 deg of lateral yaw; the remaining ~2.5 deg
is the neck-tilt zero and gravity sag, not the mount. What a simulator
consumes is the per-robot cameras_<robot>.json extrinsic, so this nominal
only seeds calibration sweeps and uncalibrated renders.

The guard test that pins the mount rotation moves with it, and the
description README's camera section gets the new provenance, the calibrated
reading as a third "still uncalibrated" item, and a fix to a stale claim that
the parked head looks level (it has been pitched since the tilt was
introduced).

Version 0.4.0 -> 0.4.1: src/ changed, and consumers pin a commit.

Co-Authored-By: Claude Fable 5.1 <noreply@anthropic.com>

File: src/manipulation_kit/description/d1/d1_wholebody.urdf (robot description, URDF)
Before this commit: robot d1_wholebody, 43 links, 42 joints
Joints:
- joint head_camera_mount: origin xyz=0.0966561 -0.0732024 -0.0282995 rpy=0 0 0.301131 -> xyz=0.0966561 -0.0732024 -0.0282995 rpy=0 0 0.261799

File: src/manipulation_kit/description/d1/d1_wholebody_gripper.urdf (robot description, URDF)
Before this commit: robot d1_wholebody_gripper, 45 links, 44 joints
Joints:
- joint head_camera_mount: origin xyz=0.0966561 -0.0732024 -0.0282995 rpy=0 0 0.301131 -> xyz=0.0966561 -0.0732024 -0.0282995 rpy=0 0 0.261799

Commit message: feat(description): guard profiles, one neck yaw, safety_zones.json deprecated
The description bundle now carries the three guard profiles a daemon
selects between, guard/profile.{d1,d1-bench,sim}.json, each with the
rule that selects it and its margins under the daemon's configuration
key names. d1 is the guard's own defaults and sim equals it. d1-bench
turns the body checks off, because a bench stand carries the two arms
with no torso, head or chassis; the arm-to-arm and same-arm checks and
every margin stay as on the robot. A test holds every profile but
d1-bench to the defaults.

The neck yaw limit has one value, +-1.5 rad (the envelope neck commands
are clamped to), in the generator, description.NECK_YAW_LIMITS_RAD and
both whole-body URDFs, instead of the vendor stop +-1.57 rad. d1.urdf
has no neck joint and is unchanged.

config/safety_zones.json describes the frozen legacy playback gate, not
the guard; it is marked deprecated (a _deprecated key and the guard
README) with its numbers unchanged.

Bundle description_version 1.1.0.

Co-Authored-By: Claude Opus 5.5 <noreply@anthropic.com>

File: src/manipulation_kit/description/d1/d1_wholebody.urdf (robot description, URDF)
Before this commit: robot d1_wholebody, 43 links, 42 joints
Joints:
- joint neck_pan: limit lower=-1.57 upper=1.57 effort=3 velocity=3.14 -> lower=-1.5 upper=1.5 effort=3 velocity=3.14

File: src/manipulation_kit/description/d1/d1_wholebody_gripper.urdf (robot description, URDF)
Before this commit: robot d1_wholebody_gripper, 45 links, 44 joints
Joints:
- joint neck_pan: limit lower=-1.57 upper=1.57 effort=3 velocity=3.14 -> lower=-1.5 upper=1.5 effort=3 velocity=3.14
