Commit message: Calibrate physical lift zero to 1293–1593 mm height range

File: src/manipulation_kit/description/d1/d1.urdf (robot description, URDF)
Before this commit: robot d1, 30 links, 29 joints
Joints:
- joint chassis_mount: origin xyz=0 0 -0.52678 rpy=0 0 0 -> xyz=0 0 -0.484 rpy=0 0 0

File: src/manipulation_kit/description/d1/d1_wholebody.urdf (robot description, URDF)
Before this commit: robot d1_wholebody, 43 links, 42 joints
Joints:
- joint lift: origin xyz=0 0 0.52678 rpy=0 0 0 -> xyz=0 0 0.484 rpy=0 0 0

File: src/manipulation_kit/description/d1/d1_wholebody_gripper.urdf (robot description, URDF)
Before this commit: robot d1_wholebody_gripper, 45 links, 44 joints
Joints:
- joint lift: origin xyz=0 0 0.52678 rpy=0 0 0 -> xyz=0 0 0.484 rpy=0 0 0

Commit message: Vendor arm inertials, and the head-camera tilt as a hardware revision
Both of these were robot facts that consumers had to reinstate after loading
a description from this package, which means the package was not saying them.

Arm links carried the family's 0.5 kg / 1e-3 diagonal placeholder while the
vendor D1 arm URDFs committed at description/d1_arm/{left,right} held the CAD
masses, COMs and tensors all along. The generator now reads them from those
files and emits them verbatim; one side of the arm chain goes from 4.05 kg of
placeholder to the vendor's 8.08 kg. TCP_Link is massless in the vendor files
and is massless here now too: it is a frame, not a part.

The head-camera mount tilt is a property of the head PART. d1-1..d1-3 wear the
15 deg part by design and the next units are built at 20 deg, so the value is
a named hardware revision (HEAD_CAMERA_TILT_DEG, head_camera_tilt_deg(),
mkit-urdf build --hardware-revision) instead of a literal in the generator.
The committed URDFs are rev1 and their head_camera_mount is unchanged. A
per-robot ArUco deviation is still not this number and belongs in that robot's
cameras_<robot>.json as an absolute head_link -> camera extrinsic.

File: src/manipulation_kit/description/d1/d1.urdf (robot description, URDF)
Before this commit: robot d1, 30 links, 29 joints
Links:
- link Base_L: mass 0.5 -> 0.8553322
- link Base_R: mass 0.5 -> 0.8553322
- link Link1_L: mass 0.5 -> 1.537551
- link Link1_R: mass 0.5 -> 1.537551
- link Link2_L: mass 0.5 -> 1.58697
- link Link2_R: mass 0.5 -> 1.58697
- link Link3_L: mass 0.5 -> 1.2915
- link Link3_R: mass 0.5 -> 1.2915
- link Link4_L: mass 0.5 -> 1.03775
- link Link4_R: mass 0.5 -> 1.03775
- link Link5_L: mass 0.5 -> 1.000479
- link Link5_R: mass 0.5 -> 1.000479
- link Link6_L: mass 0.5 -> 0.3906229
- link Link6_R: mass 0.5 -> 0.3906229
- link Link7_L: mass 0.5 -> 0.37939
- link Link7_R: mass 0.5 -> 0.37939
- link TCP_Link_L: mass 0.05 -> 0
- link TCP_Link_R: mass 0.05 -> 0

File: src/manipulation_kit/description/d1/d1_wholebody.urdf (robot description, URDF)
Before this commit: robot d1_wholebody, 43 links, 42 joints
Links:
- link Base_L: mass 0.5 -> 0.8553322
- link Base_R: mass 0.5 -> 0.8553322
- link Link1_L: mass 0.5 -> 1.537551
- link Link1_R: mass 0.5 -> 1.537551
- link Link2_L: mass 0.5 -> 1.58697
- link Link2_R: mass 0.5 -> 1.58697
- link Link3_L: mass 0.5 -> 1.2915
- link Link3_R: mass 0.5 -> 1.2915
- link Link4_L: mass 0.5 -> 1.03775
- link Link4_R: mass 0.5 -> 1.03775
- link Link5_L: mass 0.5 -> 1.000479
- link Link5_R: mass 0.5 -> 1.000479
- link Link6_L: mass 0.5 -> 0.3906229
- link Link6_R: mass 0.5 -> 0.3906229
- link Link7_L: mass 0.5 -> 0.37939
- link Link7_R: mass 0.5 -> 0.37939
- link TCP_Link_L: mass 0.05 -> 0
- link TCP_Link_R: mass 0.05 -> 0

File: src/manipulation_kit/description/d1/d1_wholebody_gripper.urdf (robot description, URDF)
Before this commit: robot d1_wholebody_gripper, 45 links, 44 joints
Links:
- link Base_L: mass 0.5 -> 0.8553322
- link Base_R: mass 0.5 -> 0.8553322
- link Link1_L: mass 0.5 -> 1.537551
- link Link1_R: mass 0.5 -> 1.537551
- link Link2_L: mass 0.5 -> 1.58697
- link Link2_R: mass 0.5 -> 1.58697
- link Link3_L: mass 0.5 -> 1.2915
- link Link3_R: mass 0.5 -> 1.2915
- link Link4_L: mass 0.5 -> 1.03775
- link Link4_R: mass 0.5 -> 1.03775
- link Link5_L: mass 0.5 -> 1.000479
- link Link5_R: mass 0.5 -> 1.000479
- link Link6_L: mass 0.5 -> 0.3906229
- link Link6_R: mass 0.5 -> 0.3906229
- link Link7_L: mass 0.5 -> 0.37939
- link Link7_R: mass 0.5 -> 0.37939
- link TCP_Link_L: mass 0.05 -> 0
- link TCP_Link_R: mass 0.05 -> 0
