Commit message: Extend the moving lift column by 53.83 mm to match the measured D1 upper body
The D1's lift telescopes: a fixed lower section on the AMR, and a moving
cover that carries the torso, both arms and the neck. Every height in this
description came from CAD that models that cover SHORTER than the built
robot, so the whole upper body sat 53.829712 mm too low.

Measured on the physical D1 (Shu, 2026-09-13): at the real 0.201 m lift and
the SDK HOME arm pose, the lowest point of the complete open gripper
assembly — including the wrist-camera plate, which is what actually reaches
lowest — clears an 884 mm wagon top by 20 mm, i.e. sits at 904 mm above the
floor. This model put it at 850.170 mm.

The correction is applied where the hardware has it: the cover gets longer
at its TOP. The lift joint origin stays at the actuator zero (0.484 m), its
0…0.300 m travel is untouched, and the cover's bottom lip stays 0.563 m
above the floor at full down — 11 mm clear of the fixed AMR cover, exactly
as before. Raising the joint origin instead reproduces the same gripper
height but opens that gap to 64.8 mm and moves a number hardware owns;
d1-isaaclab tried it (PR #42) and replaced it with this (PR #43, d5a71ec),
which is the geometry that repo ships and builds from this file.

Everything the cover carries rides up by one constant in the generator:
arm mounts 0.50 → 0.553829712, neck_pan 0.621 → 0.674829712, the chest and
back-fisheye camera mounts, the torso boxes and the static head keep-out.
The vendor body solve carries it too, so the head-camera frame — which is
SOLVED from those meshes — stays exactly where it was relative to the head.
torso_core keeps its lower bound: it is the keep-out the C++/JS validators
mirror, and a keep-out may grow but must not silently shrink.

Consumers updated in step: MotionGuard's per-arm chest keep-out (defined
relative to the shoulders, so it rides with them — the elbow-into-chest
rejection is unchanged), the d1_yubi assembler, and the pinned FK numbers.
config/safety_zones.json and the frozen safety_zones.h are deliberately NOT
re-expressed: every number they author is shoulder-relative and the whole
set moved together, so no validator's verdict changes; docs/reference/
README.md records why and what a coordinated re-expression would involve.

The one visual that an offset cannot express — the cover mesh itself, whose
lip stays while its walls lengthen — is derived by the new
description/d1/tools/extend_lift_column.py, which `mkit-urdf fetch-visuals`
now runs.

tests/test_lift_column_extension.py pins the measurement (0.904 ± 0.003 m
from the URDF's own collision geometry), agreement with d1-isaaclab's head
chain to 0.01 mm, the unchanged full-down clearance and actuator zero, and
the four copies of the constant against each other.

Co-Authored-By: Claude Fable 5.1 <noreply@anthropic.com>

File: src/manipulation_kit/description/d1/d1.urdf (robot description, URDF)
Before this commit: robot d1, 30 links, 29 joints
Links:
- link torso_column: geometry collision box size=0.0323 0.119 0.119; collision box size=0.09 0.11 0.54383
Joints:
- joint mount_L: origin xyz=0 -0.037 0.5 rpy=1.5708 0 0 -> xyz=0 -0.037 0.55383 rpy=1.5708 0 0
- joint mount_R: origin xyz=0 0.037 0.5 rpy=-1.5708 0 0 -> xyz=0 0.037 0.55383 rpy=-1.5708 0 0

File: src/manipulation_kit/description/d1/d1_wholebody.urdf (robot description, URDF)
Before this commit: robot d1_wholebody, 43 links, 42 joints
Links:
- link torso_column: geometry collision box size=0.0323 0.119 0.119; collision box size=0.09 0.11 0.54383
Joints:
- joint back_fisheye_mount: origin xyz=-0.1093 0.0015 0.4822 rpy=0 0 3.14159 -> xyz=-0.1093 0.0015 0.53603 rpy=0 0 3.14159
- joint chest_camera_mount: origin xyz=0.0891 0.0002 0.5653 rpy=0 -0.245367 0 -> xyz=0.0891 0.0002 0.61913 rpy=0 -0.245367 0
- joint mount_L: origin xyz=0 -0.037 0.5 rpy=1.5708 0 0 -> xyz=0 -0.037 0.55383 rpy=1.5708 0 0
- joint mount_R: origin xyz=0 0.037 0.5 rpy=-1.5708 0 0 -> xyz=0 0.037 0.55383 rpy=-1.5708 0 0
- joint neck_pan: origin xyz=0.0016171 0 0.621 rpy=0 0 0 -> xyz=0.0016171 0 0.67483 rpy=0 0 0

File: src/manipulation_kit/description/d1/d1_wholebody_gripper.urdf (robot description, URDF)
Before this commit: robot d1_wholebody_gripper, 45 links, 44 joints
Links:
- link torso_column: geometry collision box size=0.0323 0.119 0.119; collision box size=0.09 0.11 0.54383
Joints:
- joint back_fisheye_mount: origin xyz=-0.1093 0.0015 0.4822 rpy=0 0 3.14159 -> xyz=-0.1093 0.0015 0.53603 rpy=0 0 3.14159
- joint chest_camera_mount: origin xyz=0.0891 0.0002 0.5653 rpy=0 -0.245367 0 -> xyz=0.0891 0.0002 0.61913 rpy=0 -0.245367 0
- joint mount_L: origin xyz=0 -0.037 0.5 rpy=1.5708 0 0 -> xyz=0 -0.037 0.55383 rpy=1.5708 0 0
- joint mount_R: origin xyz=0 0.037 0.5 rpy=-1.5708 0 0 -> xyz=0 0.037 0.55383 rpy=-1.5708 0 0
- joint neck_pan: origin xyz=0.0016171 0 0.621 rpy=0 0 0 -> xyz=0.0016171 0 0.67483 rpy=0 0 0

File: src/manipulation_kit/description/d1_yubi_description_v2/urdf/d1_yubi.urdf (robot description, URDF)
Before this commit: robot d1_yubi, 28 links, 27 joints
Links:
- link torso_column: geometry visual box size=0.09 0.11 0.55383; visual cylinder length=0.085 radius=0.045
Joints:
- joint mount_L: origin xyz=0 -0.037 0.50 rpy=1.5708 0 0 -> xyz=0 -0.037 0.55383 rpy=1.5708 0 0
- joint mount_R: origin xyz=0 0.037 0.50 rpy=-1.5708 0 0 -> xyz=0 0.037 0.55383 rpy=-1.5708 0 0

Commit message: Raise the D1 upper body 29 mm at the lift origin (AMR cover height)
Replaces this branch's earlier correction — a 53.83 mm extension of the
moving lift column — with a 29 mm offset at the lift joint origin.

Shu measured d1-3 with a tape on 2026-09-16, at lift 0, floor-referenced.
The robot stands 132.2 cm to the top of its head where the spec says
129.3 cm, and the 3 cm appears at the top of the AMR: the built cover is
taller than the CAD, so everything the lift carries starts higher and the
upper body itself keeps its shape. Four frames spanning 660 mm, in mm:

    frame                      URDF (main)  measured  URDF now  residual
    torso body bottom               660       700       689      -11
    torso top                      1080.6    1120      1109.6    -10
    head RealSense (head_camera)   1233.7    1266      1262.7     -3
    head top                       1293      1322      1318.9     -3

Flat residuals across that span are what a single offset at the base looks
like. The 53.83 mm column extension gives 714 / 1134 / 1287 / 1347 —
+14…+27 mm and rising with height — because it was fitted to one
gripper-clearance reading (2026-09-13) rather than to the body. That
reading and this one disagree by ~25 mm; four frames beat one.

So the correction is applied where the hardware has it and where a single
number can express it: base_footprint -> dual_base, 0.484 -> 0.513 m.
Everything inside the dual_base frame reverts to the CAD it was measured
from — arm mounts at 0.50, neck_pan at 0.621, both torso cameras, the
torso boxes and the static head keep-out — and the lift keeps its
0…0.300 m travel. Consequently NOTHING expressed relative to the
shoulders changes: the guard's chest keep-out, config/safety_zones.json,
the frozen safety_zones.h and every IK result are bit-for-bit what main
has. Only the robot's height above the floor moved.

What that removes, versus the previous approach: the per-mount offsets,
the four hand-kept copies of the constant (generator, YUBI assembler,
guard, mesh tool), the derived torso_column_white_extended.obj and the
extend_lift_column.py that wrote it, and the fetch-visuals hook that ran
it. The generator is again the single author of the number, now named
AMR_COVER_HEIGHT_OFFSET because that is what it is.

The chassis boxes are deliberately untouched: they are authored
floor-relative and model the CAD cover, whose keep-out top (0.4987 m) is
still above the 0.460 m deck the tape found, so they stay conservative.

tests/test_lift_column_extension.py becomes
tests/test_lift_origin_amr_cover_offset.py and pins the new placement:
the lift origin at 0.513 with its travel intact, every CAD origin inside
dual_base unmoved, the zero-config world heights (Link1_R 1.013,
TCP_Link_R (0, 0.8106, 1.013), head_camera_link 1.2627), the head camera
against the tape, the chassis still on the floor, and the generator as
the only place a height correction is written down.

Co-Authored-By: Claude Fable 5.1 <noreply@anthropic.com>

File: src/manipulation_kit/description/d1/d1.urdf (robot description, URDF)
Before this commit: robot d1, 30 links, 29 joints
Links:
- link torso_column: geometry collision box size=0.0323 0.119 0.119; collision box size=0.09 0.11 0.49
Joints:
- joint chassis_mount: origin xyz=0 0 -0.484 rpy=0 0 0 -> xyz=0 0 -0.513 rpy=0 0 0
- joint mount_L: origin xyz=0 -0.037 0.55383 rpy=1.5708 0 0 -> xyz=0 -0.037 0.5 rpy=1.5708 0 0
- joint mount_R: origin xyz=0 0.037 0.55383 rpy=-1.5708 0 0 -> xyz=0 0.037 0.5 rpy=-1.5708 0 0

File: src/manipulation_kit/description/d1/d1_wholebody.urdf (robot description, URDF)
Before this commit: robot d1_wholebody, 43 links, 42 joints
Links:
- link torso_column: geometry collision box size=0.0323 0.119 0.119; collision box size=0.09 0.11 0.49
Joints:
- joint back_fisheye_mount: origin xyz=-0.1093 0.0015 0.53603 rpy=0 0 3.14159 -> xyz=-0.1093 0.0015 0.4822 rpy=0 0 3.14159
- joint chest_camera_mount: origin xyz=0.0891 0.0002 0.61913 rpy=0 -0.245367 0 -> xyz=0.0891 0.0002 0.5653 rpy=0 -0.245367 0
- joint lift: origin xyz=0 0 0.484 rpy=0 0 0 -> xyz=0 0 0.513 rpy=0 0 0
- joint mount_L: origin xyz=0 -0.037 0.55383 rpy=1.5708 0 0 -> xyz=0 -0.037 0.5 rpy=1.5708 0 0
- joint mount_R: origin xyz=0 0.037 0.55383 rpy=-1.5708 0 0 -> xyz=0 0.037 0.5 rpy=-1.5708 0 0
- joint neck_pan: origin xyz=0.0016171 0 0.67483 rpy=0 0 0 -> xyz=0.0016171 0 0.621 rpy=0 0 0

File: src/manipulation_kit/description/d1/d1_wholebody_gripper.urdf (robot description, URDF)
Before this commit: robot d1_wholebody_gripper, 45 links, 44 joints
Links:
- link torso_column: geometry collision box size=0.0323 0.119 0.119; collision box size=0.09 0.11 0.49
Joints:
- joint back_fisheye_mount: origin xyz=-0.1093 0.0015 0.53603 rpy=0 0 3.14159 -> xyz=-0.1093 0.0015 0.4822 rpy=0 0 3.14159
- joint chest_camera_mount: origin xyz=0.0891 0.0002 0.61913 rpy=0 -0.245367 0 -> xyz=0.0891 0.0002 0.5653 rpy=0 -0.245367 0
- joint lift: origin xyz=0 0 0.484 rpy=0 0 0 -> xyz=0 0 0.513 rpy=0 0 0
- joint mount_L: origin xyz=0 -0.037 0.55383 rpy=1.5708 0 0 -> xyz=0 -0.037 0.5 rpy=1.5708 0 0
- joint mount_R: origin xyz=0 0.037 0.55383 rpy=-1.5708 0 0 -> xyz=0 0.037 0.5 rpy=-1.5708 0 0
- joint neck_pan: origin xyz=0.0016171 0 0.67483 rpy=0 0 0 -> xyz=0.0016171 0 0.621 rpy=0 0 0

File: src/manipulation_kit/description/d1_yubi_description_v2/urdf/d1_yubi.urdf (robot description, URDF)
Before this commit: robot d1_yubi, 28 links, 27 joints
Links:
- link torso_column: geometry visual box size=0.09 0.11 0.50; visual cylinder length=0.085 radius=0.045
Joints:
- joint mount_L: origin xyz=0 -0.037 0.55383 rpy=1.5708 0 0 -> xyz=0 -0.037 0.50 rpy=1.5708 0 0
- joint mount_R: origin xyz=0 0.037 0.55383 rpy=-1.5708 0 0 -> xyz=0 0.037 0.50 rpy=-1.5708 0 0

Commit message: feat(guard)!: rounded belly band and the hand envelope in the body check
The measured torso box stood ~40 mm proud of the shell at the front
obliques, where the shell curves inward, so the arm stopped short there;
and every body distal of the flange was excluded from the checks, so the
gripper's jaw tips could reach the belly while the arm links reported
clearance.

- torso_belly keeps its measured faces and gets rounded vertical edges
  (front 80 mm, back 40 mm), fitted to the CAD shell outline moved onto
  the measured faces: the shell is at most 3.4 mm outside the shape and
  the air covered at the front corners drops from 39.8 to 7.6 mm
  (description/d1/tools/fit_torso_belly.py). In URDF it is the exact
  union of three boxes and four vertical cylinders; the guard gains
  vertical body cylinders (convex golden-section distance, pruned by the
  part of each cylinder the body's boxes leave uncovered) and names every
  part by its body.
- d1.urdf carries hand_envelope_<R|L>: six capsules covering every
  collision box of the parallel-gripper description (jaws over their
  whole travel, camera plate and housing) to within 0.74 mm. They are
  checked against the body shapes, the chest keep-out and the other
  arm's structure at the body margin; not against their own arm, the
  other hand, or scene obstacles.

Co-Authored-By: Claude Fable 5.1 <noreply@anthropic.com>

File: src/manipulation_kit/description/d1/d1.urdf (robot description, URDF)
Before this commit: robot d1, 30 links, 29 joints
Links:
- added link hand_envelope_L, mass 1e-06; collision cylinder length=0.028 radius=0.03; collision cylinder length=0.032 radius=0.043
- added link hand_envelope_R, mass 1e-06; collision cylinder length=0.028 radius=0.03; collision cylinder length=0.032 radius=0.043
- link torso_column: geometry collision box size=0.0323 0.119 0.119; collision box size=0.04 0.14 0.25
Joints:
- added joint hand_envelope_L_mount: type fixed, parent TCP_Link_L, child hand_envelope_L, origin xyz=0 0 0 rpy=0 0 0
- added joint hand_envelope_R_mount: type fixed, parent TCP_Link_R, child hand_envelope_R, origin xyz=0 0 0 rpy=0 0 3.14159

File: src/manipulation_kit/description/d1/d1_wholebody.urdf (robot description, URDF)
Before this commit: robot d1_wholebody, 43 links, 42 joints
Links:
- link torso_column: geometry collision box size=0.0323 0.119 0.119; collision box size=0.04 0.14 0.25

File: src/manipulation_kit/description/d1/d1_wholebody_gripper.urdf (robot description, URDF)
Before this commit: robot d1_wholebody_gripper, 45 links, 44 joints
Links:
- link torso_column: geometry collision box size=0.0323 0.119 0.119; collision box size=0.04 0.14 0.25
