Commit message: feat(description): rename the stand model d1-arms-stand; no end effector
Robot model ids name the kinematic structure, never a use, a site or an
end effector: `<platform>` for a whole robot, `<platform>-<parts>-<mount>`
for parts on something else. `arm-ee-bench` becomes `d1-arms-stand`
(URDFs d1_arms_stand.urdf and d1_arms_stand_visual.urdf, export variant,
guard profile and lock of the same name, description_version 1.0.0).

The stand's URDFs carry no end effector and no hand envelope: the arms end
at their flanges, and the guard checks arm against arm, each arm against
itself and the joint limits only. robot.json states it in
end_effectors.collision_checked (false on the stand, true on d1), and
states whether recorded or synthetic input may drive the real arms in
recorded_input (operator_override on the stand, refused on d1). The d1
bundle moves to 1.4.0. Version 0.22.8.

Co-Authored-By: Claude Opus 5.5 <noreply@anthropic.com>
Claude-Session: https://claude.ai/code/session_01MPdyHzyk4wQqHzwgS78FVb

File: src/manipulation_kit/description/d1/d1_arms_stand.urdf (robot description, URDF)
Before this commit: robot arm_ee_bench, 24 links, 23 joints
Links:
- removed link hand_envelope_L
- removed link hand_envelope_R
- removed link wujihand2_L
- removed link wujihand2_R
Joints:
- removed joint hand_envelope_L_mount
- removed joint hand_envelope_R_mount
- removed joint wujihand2_L_mount
- removed joint wujihand2_R_mount

File: src/manipulation_kit/description/d1/d1_arms_stand_visual.urdf (robot description, URDF)
Before this commit: robot arm_ee_bench_visual, 24 links, 23 joints
Links:
- removed link hand_envelope_L
- removed link hand_envelope_R
- removed link wujihand2_L
- removed link wujihand2_R
Joints:
- removed joint hand_envelope_L_mount
- removed joint hand_envelope_R_mount
- removed joint wujihand2_L_mount
- removed joint wujihand2_R_mount
