Commit message: Refresh whole-body export for rear panel visuals

File: dist/d1-wholebody-gripper/d1_wholebody_gripper.urdf (robot description, URDF)
Before this commit: robot d1_wholebody_gripper, 45 links, 44 joints
Links:
- link chassis_link: geometry collision box size=0.14 0.14 0.5; collision box size=0.5395 0.4805 0.223
- link torso_column: geometry collision box size=0.0323 0.119 0.119; collision box size=0.09 0.11 0.49

Commit message: Refresh maintained whole-body export with corrected head and controls

File: dist/d1-wholebody-gripper/d1_wholebody_gripper.urdf (robot description, URDF)
Before this commit: robot d1_wholebody_gripper, 45 links, 44 joints
Links:
- link chassis_link: geometry collision box size=0.14 0.14 0.5; collision box size=0.5395 0.4805 0.223
- link head_link: geometry collision box size=0.2008 0.185 0.19; visual mesh filename=meshes/body_hifi/head_link_cyan.obj
- link torso_column: geometry collision box size=0.0323 0.119 0.119; collision box size=0.09 0.11 0.49

Commit message: Refresh whole-body export for gallery-refined chassis and optics

File: dist/d1-wholebody-gripper/d1_wholebody_gripper.urdf (robot description, URDF)
Before this commit: robot d1_wholebody_gripper, 45 links, 44 joints
Links:
- link chassis_link: geometry collision box size=0.14 0.14 0.5; collision box size=0.5395 0.4805 0.223
- link head_link: geometry collision box size=0.2008 0.185 0.19; visual mesh filename=meshes/body_hifi/head_link_cyan.obj

Commit message: Refresh whole-body export for calibrated physical lift zero

File: dist/d1-wholebody-gripper/d1_wholebody_gripper.urdf (robot description, URDF)
Before this commit: robot d1_wholebody_gripper, 45 links, 44 joints
Joints:
- joint lift: origin xyz=0 0 0.52678 rpy=0 0 0 -> xyz=0 0 0.484 rpy=0 0 0

Commit message: Re-export the prebuilt dist/ artifacts for the new arm inertials

File: dist/d1-wholebody-gripper/d1_wholebody_gripper.urdf (robot description, URDF)
Before this commit: robot d1_wholebody_gripper, 45 links, 44 joints
Links:
- link Base_L: mass 0.5 -> 0.8553322
- link Base_R: mass 0.5 -> 0.8553322
- link Link1_L: mass 0.5 -> 1.537551
- link Link1_R: mass 0.5 -> 1.537551
- link Link2_L: mass 0.5 -> 1.58697
- link Link2_R: mass 0.5 -> 1.58697
- link Link3_L: mass 0.5 -> 1.2915
- link Link3_R: mass 0.5 -> 1.2915
- link Link4_L: mass 0.5 -> 1.03775
- link Link4_R: mass 0.5 -> 1.03775
- link Link5_L: mass 0.5 -> 1.000479
- link Link5_R: mass 0.5 -> 1.000479
- link Link6_L: mass 0.5 -> 0.3906229
- link Link6_R: mass 0.5 -> 0.3906229
- link Link7_L: mass 0.5 -> 0.37939
- link Link7_R: mass 0.5 -> 0.37939
- link TCP_Link_L: mass 0.05 -> 0
- link TCP_Link_R: mass 0.05 -> 0
