Commit message: Re-export dist/ with the extended lift column
Regenerated with `mkit-urdf export d1-collision|d1-wholebody-gripper`, so the
vendored copies carry the measured cover extension and the whole-body export
declares the derived cover mesh (torso_column_white_extended.obj) in its
absent-optional list.

Co-Authored-By: Claude Fable 5.1 <noreply@anthropic.com>

File: dist/d1-wholebody-gripper/d1_wholebody_gripper.urdf (robot description, URDF)
Before this commit: robot d1_wholebody_gripper, 45 links, 44 joints
Links:
- link torso_column: geometry collision box size=0.0323 0.119 0.119; collision box size=0.09 0.11 0.54383
Joints:
- joint back_fisheye_mount: origin xyz=-0.1093 0.0015 0.4822 rpy=0 0 3.14159 -> xyz=-0.1093 0.0015 0.53603 rpy=0 0 3.14159
- joint chest_camera_mount: origin xyz=0.0891 0.0002 0.5653 rpy=0 -0.245367 0 -> xyz=0.0891 0.0002 0.61913 rpy=0 -0.245367 0
- joint mount_L: origin xyz=0 -0.037 0.5 rpy=1.5708 0 0 -> xyz=0 -0.037 0.55383 rpy=1.5708 0 0
- joint mount_R: origin xyz=0 0.037 0.5 rpy=-1.5708 0 0 -> xyz=0 0.037 0.55383 rpy=-1.5708 0 0
- joint neck_pan: origin xyz=0.0016171 0 0.621 rpy=0 0 0 -> xyz=0.0016171 0 0.67483 rpy=0 0 0

Commit message: Re-export dist/ on the 29 mm lift origin
Regenerated with `mkit-urdf export d1-collision|d1-wholebody-gripper`, so the
vendored copies carry the measured AMR cover offset. Against main each export
differs by exactly one line — the lift joint origin (0.484 -> 0.513 m), and
the chassis mount that mirrors it in the collision variant — and the
whole-body export's absent-optional list is back to the plain CAD column mesh
now that the derived torso_column_white_extended.obj is gone.

Co-Authored-By: Claude Fable 5.1 <noreply@anthropic.com>

File: dist/d1-wholebody-gripper/d1_wholebody_gripper.urdf (robot description, URDF)
Before this commit: robot d1_wholebody_gripper, 45 links, 44 joints
Links:
- link torso_column: geometry collision box size=0.0323 0.119 0.119; collision box size=0.09 0.11 0.49
Joints:
- joint back_fisheye_mount: origin xyz=-0.1093 0.0015 0.53603 rpy=0 0 3.14159 -> xyz=-0.1093 0.0015 0.4822 rpy=0 0 3.14159
- joint chest_camera_mount: origin xyz=0.0891 0.0002 0.61913 rpy=0 -0.245367 0 -> xyz=0.0891 0.0002 0.5653 rpy=0 -0.245367 0
- joint lift: origin xyz=0 0 0.484 rpy=0 0 0 -> xyz=0 0 0.513 rpy=0 0 0
- joint mount_L: origin xyz=0 -0.037 0.55383 rpy=1.5708 0 0 -> xyz=0 -0.037 0.5 rpy=1.5708 0 0
- joint mount_R: origin xyz=0 0.037 0.55383 rpy=-1.5708 0 0 -> xyz=0 0.037 0.5 rpy=-1.5708 0 0
- joint neck_pan: origin xyz=0.0016171 0 0.67483 rpy=0 0 0 -> xyz=0.0016171 0 0.621 rpy=0 0 0

Commit message: Re-export dist/ on the 15 deg head-camera pitch
Regenerated with `mkit-urdf export d1-collision|d1-wholebody-gripper`. The
whole-body export differs by exactly one line — head_camera_mount rpy,
0.301131 -> 0.261799 — and d1-collision only restamps its source commit,
since the guard model carries no cameras.

Co-Authored-By: Claude Fable 5.1 <noreply@anthropic.com>

File: dist/d1-wholebody-gripper/d1_wholebody_gripper.urdf (robot description, URDF)
Before this commit: robot d1_wholebody_gripper, 45 links, 44 joints
Joints:
- joint head_camera_mount: origin xyz=0.0966561 -0.0732024 -0.0282995 rpy=0 0 0.301131 -> xyz=0.0966561 -0.0732024 -0.0282995 rpy=0 0 0.261799

Commit message: chore(dist): re-export d1-collision and d1-wholebody-gripper from the rounded-belly commit
Co-Authored-By: Claude Fable 5.1 <noreply@anthropic.com>

File: dist/d1-wholebody-gripper/d1_wholebody_gripper.urdf (robot description, URDF)
Before this commit: robot d1_wholebody_gripper, 45 links, 44 joints
Links:
- link torso_column: geometry collision box size=0.0323 0.119 0.119; collision box size=0.04 0.14 0.25

Commit message: chore(description): regenerate the whole-body export, accept the deprecation key
The vendored dist/d1-wholebody-gripper export follows the neck yaw limit
change, and the safety_zones.json export check accepts its _deprecated
metadata key alongside the existing comment keys.

Co-Authored-By: Claude Opus 5.5 <noreply@anthropic.com>

File: dist/d1-wholebody-gripper/d1_wholebody_gripper.urdf (robot description, URDF)
Before this commit: robot d1_wholebody_gripper, 45 links, 44 joints
Joints:
- joint neck_pan: limit lower=-1.57 upper=1.57 effort=3 velocity=3.14 -> lower=-1.5 upper=1.5 effort=3 velocity=3.14
