Commit message: Start the torso keep-out at the moving sleeve's lip
torso_core ran the full 0..0.49 m of torso_column, from the lift origin up.
The bottom 79 mm is not torso: with the lift retracted the sleeve's lower lip
sits at world z 0.592 m against a lift origin of 0.513 m (measured on d1-3 in
the d1-isaaclab ustea physical-mount check), so that band is the fixed column,
and it lies inside the chassis-side lift_pole box (X +/-70, Y -67..73, world
z 0.389..0.889) which encloses torso_core's X +/-45 / Y +/-55 footprint.

torso_core now spans z 0.079..0.49 (TORSO_SLEEVE_LIP_M). The guard loses no
keep-out at q_lift = 0; at full 0.30 m extension the top 3 mm of the removed
band are covered by no box. Every simulator that loaded the old box saw it
collide with the AMR cover; d1-isaaclab carried a local carve for exactly
this. Shu approved shrinking the keep-out on 2026-09-20.

d1-firmware's Rust guard mirrors this box from the URDF and pins it with
golden vectors; its kit pin bump needs gen_guard_vectors.py re-run.

File: dist/d1-collision/d1.urdf (robot description, URDF)
Before this commit: robot d1, 30 links, 29 joints
Links:
- link torso_column: geometry collision box size=0.0323 0.119 0.119; collision box size=0.09 0.11 0.411

File: dist/d1-wholebody-gripper/d1_wholebody_gripper.urdf (robot description, URDF)
Before this commit: robot d1_wholebody_gripper, 45 links, 44 joints
Links:
- link torso_column: geometry collision box size=0.0323 0.119 0.119; collision box size=0.09 0.11 0.411

File: src/manipulation_kit/description/d1/d1_wholebody.urdf (robot description, URDF)
Before this commit: robot d1_wholebody, 43 links, 42 joints
Links:
- link torso_column: geometry collision box size=0.0323 0.119 0.119; collision box size=0.09 0.11 0.411

File: src/manipulation_kit/description/d1/d1_wholebody_gripper.urdf (robot description, URDF)
Before this commit: robot d1_wholebody_gripper, 45 links, 44 joints
Links:
- link torso_column: geometry collision box size=0.0323 0.119 0.119; collision box size=0.09 0.11 0.411
