Commit message: feat(guard)!: fit the arm capsules to the vendor meshes, measured torso box, exact distance, 5 mm margin
The guard's arm model was one hand-picked capsule per link, up to 23 mm
thinner than the vendor meshes; the torso box came from the CAD shell,
20 mm wider than the built robot and 8 mm short at the front, with its top
in the shoulder sleeve; and segment-to-box distance was sampled at 25
points (up to ~2.4 mm optimistic). The 30/60 mm margins compensated.

- ARM_CAPSULES: per link a tube and a housing capsule fitted by the new
  tools/fit_arm_capsules.py so that every vertex of both arms' meshes is
  inside; record in description/d1/arm_capsule_fit.json, checked by
  tests/guard/test_arm_capsule_fit.py (always against the record, and
  against the meshes when MKIT_ASSETS_DIR is set).
- torso_belly: x -0.130..0.135, y +/-0.110 (measured on the robot), z top
  0.44 where the CAD shell becomes the shoulder sleeve; the exempt shell and
  the chest keep-out start at 0.44.
- Link1 is body-exempt like Base (its capsules do not move with any joint).
- seg_aabb_distance is exact.
- Default margins: body 0.005 m, arm-arm 0.035 m (keeps grippers side by
  side passing from ~140 mm, as 0.06 did on the old radii).

HOME: 31.7 mm from torso_belly (was 30.3 against a 30 mm margin); the arm
hanging at the side passes; arms crossed at the chest are refused
(tests/guard/test_guard_postures.py). URDFs and dist/ regenerated.
Version 0.15.0.

Co-Authored-By: Claude Opus 5.5 (1M context) <noreply@anthropic.com>

File: dist/d1-collision/d1.urdf (robot description, URDF)
Before this commit: robot d1, 30 links, 29 joints
Links:
- link Base_L: geometry collision cylinder length=0.1586 radius=0.0566; collision sphere radius=0.0566
- link Base_R: geometry collision cylinder length=0.1586 radius=0.0566; collision sphere radius=0.0566
- link Link1_L: geometry collision cylinder length=0.108 radius=0.0495; collision sphere radius=0.0495
- link Link1_R: geometry collision cylinder length=0.108 radius=0.0495; collision sphere radius=0.0495
- link Link2_L: geometry collision cylinder length=0.08 radius=0.0572; collision sphere radius=0.0572
- link Link2_R: geometry collision cylinder length=0.08 radius=0.0572; collision sphere radius=0.0572
- link Link3_L: geometry collision cylinder length=0.02 radius=0.0487; collision cylinder length=0.1116 radius=0.043
- link Link3_R: geometry collision cylinder length=0.02 radius=0.0487; collision cylinder length=0.1116 radius=0.043
- link Link4_L: geometry collision cylinder length=0.053621 radius=0.059; collision sphere radius=0.059
- link Link4_R: geometry collision cylinder length=0.053621 radius=0.059; collision sphere radius=0.059
- link Link5_L: geometry collision cylinder length=0.06 radius=0.0232; collision cylinder length=0.1179 radius=0.0499
- link Link5_R: geometry collision cylinder length=0.06 radius=0.0232; collision cylinder length=0.1179 radius=0.0499
- link Link6_L: geometry collision cylinder length=0.005 radius=0.0368; collision cylinder length=0.04 radius=0.0339
- link Link6_R: geometry collision cylinder length=0.005 radius=0.0368; collision cylinder length=0.04 radius=0.0339
- link Link7_L: geometry collision cylinder length=0.037 radius=0.0442; collision sphere radius=0.0442
- link Link7_R: geometry collision cylinder length=0.037 radius=0.0442; collision sphere radius=0.0442
- link torso_column: geometry collision box size=0.0323 0.119 0.119; collision box size=0.09 0.11 0.411

File: dist/d1-wholebody-gripper/d1_wholebody_gripper.urdf (robot description, URDF)
Before this commit: robot d1_wholebody_gripper, 45 links, 44 joints
Links:
- link Base_L: geometry collision cylinder length=0.1586 radius=0.0566; collision sphere radius=0.0566
- link Base_R: geometry collision cylinder length=0.1586 radius=0.0566; collision sphere radius=0.0566
- link Link1_L: geometry collision cylinder length=0.108 radius=0.0495; collision sphere radius=0.0495
- link Link1_R: geometry collision cylinder length=0.108 radius=0.0495; collision sphere radius=0.0495
- link Link2_L: geometry collision cylinder length=0.08 radius=0.0572; collision sphere radius=0.0572
- link Link2_R: geometry collision cylinder length=0.08 radius=0.0572; collision sphere radius=0.0572
- link Link3_L: geometry collision cylinder length=0.02 radius=0.0487; collision cylinder length=0.1116 radius=0.043
- link Link3_R: geometry collision cylinder length=0.02 radius=0.0487; collision cylinder length=0.1116 radius=0.043
- link Link4_L: geometry collision cylinder length=0.053621 radius=0.059; collision sphere radius=0.059
- link Link4_R: geometry collision cylinder length=0.053621 radius=0.059; collision sphere radius=0.059
- link Link5_L: geometry collision cylinder length=0.06 radius=0.0232; collision cylinder length=0.1179 radius=0.0499
- link Link5_R: geometry collision cylinder length=0.06 radius=0.0232; collision cylinder length=0.1179 radius=0.0499
- link Link6_L: geometry collision cylinder length=0.005 radius=0.0368; collision cylinder length=0.04 radius=0.0339
- link Link6_R: geometry collision cylinder length=0.005 radius=0.0368; collision cylinder length=0.04 radius=0.0339
- link Link7_L: geometry collision cylinder length=0.037 radius=0.0442; collision sphere radius=0.0442
- link Link7_R: geometry collision cylinder length=0.037 radius=0.0442; collision sphere radius=0.0442
- link torso_column: geometry collision box size=0.0323 0.119 0.119; collision box size=0.09 0.11 0.411

File: src/manipulation_kit/description/d1/d1_wholebody.urdf (robot description, URDF)
Before this commit: robot d1_wholebody, 43 links, 42 joints
Links:
- link Base_L: geometry collision cylinder length=0.1586 radius=0.0566; collision sphere radius=0.0566
- link Base_R: geometry collision cylinder length=0.1586 radius=0.0566; collision sphere radius=0.0566
- link Link1_L: geometry collision cylinder length=0.108 radius=0.0495; collision sphere radius=0.0495
- link Link1_R: geometry collision cylinder length=0.108 radius=0.0495; collision sphere radius=0.0495
- link Link2_L: geometry collision cylinder length=0.08 radius=0.0572; collision sphere radius=0.0572
- link Link2_R: geometry collision cylinder length=0.08 radius=0.0572; collision sphere radius=0.0572
- link Link3_L: geometry collision cylinder length=0.02 radius=0.0487; collision cylinder length=0.1116 radius=0.043
- link Link3_R: geometry collision cylinder length=0.02 radius=0.0487; collision cylinder length=0.1116 radius=0.043
- link Link4_L: geometry collision cylinder length=0.053621 radius=0.059; collision sphere radius=0.059
- link Link4_R: geometry collision cylinder length=0.053621 radius=0.059; collision sphere radius=0.059
- link Link5_L: geometry collision cylinder length=0.06 radius=0.0232; collision cylinder length=0.1179 radius=0.0499
- link Link5_R: geometry collision cylinder length=0.06 radius=0.0232; collision cylinder length=0.1179 radius=0.0499
- link Link6_L: geometry collision cylinder length=0.005 radius=0.0368; collision cylinder length=0.04 radius=0.0339
- link Link6_R: geometry collision cylinder length=0.005 radius=0.0368; collision cylinder length=0.04 radius=0.0339
- link Link7_L: geometry collision cylinder length=0.037 radius=0.0442; collision sphere radius=0.0442
- link Link7_R: geometry collision cylinder length=0.037 radius=0.0442; collision sphere radius=0.0442
- link torso_column: geometry collision box size=0.0323 0.119 0.119; collision box size=0.09 0.11 0.411

File: src/manipulation_kit/description/d1/d1_wholebody_gripper.urdf (robot description, URDF)
Before this commit: robot d1_wholebody_gripper, 45 links, 44 joints
Links:
- link Base_L: geometry collision cylinder length=0.1586 radius=0.0566; collision sphere radius=0.0566
- link Base_R: geometry collision cylinder length=0.1586 radius=0.0566; collision sphere radius=0.0566
- link Link1_L: geometry collision cylinder length=0.108 radius=0.0495; collision sphere radius=0.0495
- link Link1_R: geometry collision cylinder length=0.108 radius=0.0495; collision sphere radius=0.0495
- link Link2_L: geometry collision cylinder length=0.08 radius=0.0572; collision sphere radius=0.0572
- link Link2_R: geometry collision cylinder length=0.08 radius=0.0572; collision sphere radius=0.0572
- link Link3_L: geometry collision cylinder length=0.02 radius=0.0487; collision cylinder length=0.1116 radius=0.043
- link Link3_R: geometry collision cylinder length=0.02 radius=0.0487; collision cylinder length=0.1116 radius=0.043
- link Link4_L: geometry collision cylinder length=0.053621 radius=0.059; collision sphere radius=0.059
- link Link4_R: geometry collision cylinder length=0.053621 radius=0.059; collision sphere radius=0.059
- link Link5_L: geometry collision cylinder length=0.06 radius=0.0232; collision cylinder length=0.1179 radius=0.0499
- link Link5_R: geometry collision cylinder length=0.06 radius=0.0232; collision cylinder length=0.1179 radius=0.0499
- link Link6_L: geometry collision cylinder length=0.005 radius=0.0368; collision cylinder length=0.04 radius=0.0339
- link Link6_R: geometry collision cylinder length=0.005 radius=0.0368; collision cylinder length=0.04 radius=0.0339
- link Link7_L: geometry collision cylinder length=0.037 radius=0.0442; collision sphere radius=0.0442
- link Link7_R: geometry collision cylinder length=0.037 radius=0.0442; collision sphere radius=0.0442
- link torso_column: geometry collision box size=0.0323 0.119 0.119; collision box size=0.09 0.11 0.411

Commit message: feat(guard)!: thin link tubes + 97 mm J2/J4 housings (Shu's shape), arm-arm 0.045
Shu, 2026-09-23: the fully covering capsules were too fat ("the links are
thinner; only the shoulder and elbow housings are 97 mm"). The arm model is
now a tube per link at the link's real tube radius plus the J2/J4
housings as radius-48.5 mm capsules on the joint axis, every capsule
trimmed so its rounded ends stop at the mesh ends.

The housing cover-plate rims and tube ends are not covered (up to 24 mm,
Link4); the per-link residual is in arm_capsule_fit.json and the mesh test
fails past residual + 1 mm. Covering them took ~200 capsules per arm and
was rejected for call rate.

HOME clears torso_belly by 45.4 mm at margin 0; arm at the side 33.2;
arms crossed refused (-14.6). Arm-arm margin 0.045 keeps side-by-side
grippers passing from ~140 mm (47.4 mm there; 135 mm refused).

Co-Authored-By: Claude Opus 5.5 (1M context) <noreply@anthropic.com>

File: dist/d1-collision/d1.urdf (robot description, URDF)
Before this commit: robot d1, 30 links, 29 joints
Links:
- link Link1_L: geometry collision cylinder length=0.088 radius=0.0556; collision sphere radius=0.0556
- link Link1_R: geometry collision cylinder length=0.088 radius=0.0556; collision sphere radius=0.0556
- link Link2_L: geometry collision cylinder length=0.0188 radius=0.0485; collision cylinder length=0.039 radius=0.0425
- link Link2_R: geometry collision cylinder length=0.0188 radius=0.0485; collision cylinder length=0.039 radius=0.0425
- link Link3_L: geometry collision cylinder length=0.0965 radius=0.0425; collision sphere radius=0.0425
- link Link3_R: geometry collision cylinder length=0.0965 radius=0.0425; collision sphere radius=0.0425
- link Link4_L: geometry collision cylinder length=0.00963328 radius=0.0465; collision cylinder length=0.0118 radius=0.0485
- link Link4_R: geometry collision cylinder length=0.00963328 radius=0.0465; collision cylinder length=0.0118 radius=0.0485
- link Link5_L: geometry collision cylinder length=0.0932 radius=0.0482; collision sphere radius=0.0482
- link Link5_R: geometry collision cylinder length=0.0932 radius=0.0482; collision sphere radius=0.0482
- link Link6_L: geometry collision cylinder length=0.0014 radius=0.0313; collision sphere radius=0.0313
- link Link6_R: geometry collision cylinder length=0.0014 radius=0.0313; collision sphere radius=0.0313
- link Link7_L: geometry collision cylinder length=0.0478 radius=0.0345; collision sphere radius=0.0345
- link Link7_R: geometry collision cylinder length=0.0478 radius=0.0345; collision sphere radius=0.0345

File: dist/d1-wholebody-gripper/d1_wholebody_gripper.urdf (robot description, URDF)
Before this commit: robot d1_wholebody_gripper, 45 links, 44 joints
Links:
- link Link1_L: geometry collision cylinder length=0.088 radius=0.0556; collision sphere radius=0.0556
- link Link1_R: geometry collision cylinder length=0.088 radius=0.0556; collision sphere radius=0.0556
- link Link2_L: geometry collision cylinder length=0.0188 radius=0.0485; collision cylinder length=0.039 radius=0.0425
- link Link2_R: geometry collision cylinder length=0.0188 radius=0.0485; collision cylinder length=0.039 radius=0.0425
- link Link3_L: geometry collision cylinder length=0.0965 radius=0.0425; collision sphere radius=0.0425
- link Link3_R: geometry collision cylinder length=0.0965 radius=0.0425; collision sphere radius=0.0425
- link Link4_L: geometry collision cylinder length=0.00963328 radius=0.0465; collision cylinder length=0.0118 radius=0.0485
- link Link4_R: geometry collision cylinder length=0.00963328 radius=0.0465; collision cylinder length=0.0118 radius=0.0485
- link Link5_L: geometry collision cylinder length=0.0932 radius=0.0482; collision sphere radius=0.0482
- link Link5_R: geometry collision cylinder length=0.0932 radius=0.0482; collision sphere radius=0.0482
- link Link6_L: geometry collision cylinder length=0.0014 radius=0.0313; collision sphere radius=0.0313
- link Link6_R: geometry collision cylinder length=0.0014 radius=0.0313; collision sphere radius=0.0313
- link Link7_L: geometry collision cylinder length=0.0478 radius=0.0345; collision sphere radius=0.0345
- link Link7_R: geometry collision cylinder length=0.0478 radius=0.0345; collision sphere radius=0.0345

File: src/manipulation_kit/description/d1/d1_wholebody.urdf (robot description, URDF)
Before this commit: robot d1_wholebody, 43 links, 42 joints
Links:
- link Link1_L: geometry collision cylinder length=0.088 radius=0.0556; collision sphere radius=0.0556
- link Link1_R: geometry collision cylinder length=0.088 radius=0.0556; collision sphere radius=0.0556
- link Link2_L: geometry collision cylinder length=0.0188 radius=0.0485; collision cylinder length=0.039 radius=0.0425
- link Link2_R: geometry collision cylinder length=0.0188 radius=0.0485; collision cylinder length=0.039 radius=0.0425
- link Link3_L: geometry collision cylinder length=0.0965 radius=0.0425; collision sphere radius=0.0425
- link Link3_R: geometry collision cylinder length=0.0965 radius=0.0425; collision sphere radius=0.0425
- link Link4_L: geometry collision cylinder length=0.00963328 radius=0.0465; collision cylinder length=0.0118 radius=0.0485
- link Link4_R: geometry collision cylinder length=0.00963328 radius=0.0465; collision cylinder length=0.0118 radius=0.0485
- link Link5_L: geometry collision cylinder length=0.0932 radius=0.0482; collision sphere radius=0.0482
- link Link5_R: geometry collision cylinder length=0.0932 radius=0.0482; collision sphere radius=0.0482
- link Link6_L: geometry collision cylinder length=0.0014 radius=0.0313; collision sphere radius=0.0313
- link Link6_R: geometry collision cylinder length=0.0014 radius=0.0313; collision sphere radius=0.0313
- link Link7_L: geometry collision cylinder length=0.0478 radius=0.0345; collision sphere radius=0.0345
- link Link7_R: geometry collision cylinder length=0.0478 radius=0.0345; collision sphere radius=0.0345

File: src/manipulation_kit/description/d1/d1_wholebody_gripper.urdf (robot description, URDF)
Before this commit: robot d1_wholebody_gripper, 45 links, 44 joints
Links:
- link Link1_L: geometry collision cylinder length=0.088 radius=0.0556; collision sphere radius=0.0556
- link Link1_R: geometry collision cylinder length=0.088 radius=0.0556; collision sphere radius=0.0556
- link Link2_L: geometry collision cylinder length=0.0188 radius=0.0485; collision cylinder length=0.039 radius=0.0425
- link Link2_R: geometry collision cylinder length=0.0188 radius=0.0485; collision cylinder length=0.039 radius=0.0425
- link Link3_L: geometry collision cylinder length=0.0965 radius=0.0425; collision sphere radius=0.0425
- link Link3_R: geometry collision cylinder length=0.0965 radius=0.0425; collision sphere radius=0.0425
- link Link4_L: geometry collision cylinder length=0.00963328 radius=0.0465; collision cylinder length=0.0118 radius=0.0485
- link Link4_R: geometry collision cylinder length=0.00963328 radius=0.0465; collision cylinder length=0.0118 radius=0.0485
- link Link5_L: geometry collision cylinder length=0.0932 radius=0.0482; collision sphere radius=0.0482
- link Link5_R: geometry collision cylinder length=0.0932 radius=0.0482; collision sphere radius=0.0482
- link Link6_L: geometry collision cylinder length=0.0014 radius=0.0313; collision sphere radius=0.0313
- link Link6_R: geometry collision cylinder length=0.0014 radius=0.0313; collision sphere radius=0.0313
- link Link7_L: geometry collision cylinder length=0.0478 radius=0.0345; collision sphere radius=0.0345
- link Link7_R: geometry collision cylinder length=0.0478 radius=0.0345; collision sphere radius=0.0345
